File: esp32-c6.kicad_pcb (KiCad board)
At the start: 2 copper layers, 78.5 x 39 mm, 75 parts, among them J1 USB_C_Receptacle_USB2.0_14P, J2 USB_C_Receptacle_USB2.0_14P, J3 54-00166, J4 Conn_01x08_Socket, J5 Conn_01x06_Socket, J6 Conn_01x04, J7 Conn_01x10_Socket, J8 Conn_01x06_Socket, Q1 BC847BDW1, SW1 SW_Push, SW2 SW_Push, U1 CP2102N-Axx-xQFN28, U2 MPQ9841GLE-5-AEC1-Z, U3 NCP1117-3.3_SOT223, U4 ESP32-C6-WROOM-1-N8

Commit message: Refinement to pcb and schematic layout
Parts:
- removed J7: Conn_01x10_Socket, Connector_PinSocket_2.00mm:PinSocket_1x10_P2.00mm_Vertical
- added J9: Conn_01x09_Socket, Connector_PinSocket_2.00mm:PinSocket_1x09_P2.00mm_Vertical, F.Cu at (171.7, 162.4)
- moved F1 4.03 mm to (200.4, 155.1), turned to -90 degrees
- moved J6 0.22 mm to (194.2, 146.9)
Routing:
- net Net-(J6-Pin_2): track 4.78 -> 9.75 mm
- net /esp32-c6 Pinout/IO11: track 30.8 -> 26.4 mm, vias 2 -> 1
- net /esp32-c6 Pinout/IO15: track 13.7 -> 9.42 mm, vias 2 -> 1
- net /esp32-c6 Pinout/IO10: track 29.0 -> 24.9 mm, vias 2 -> 1
- net +3.3V: track 144.4 -> 141.3 mm
- net GND: track 5.31 -> 7.28 mm, vias 4 -> 29
- net /esp32-c6 Pinout/IO22: track 19.5 -> 17.9 mm
- net /esp32-c6 Pinout/IO21: track 19.0 -> 17.4 mm
- net /esp32-c6 Pinout/IO19: track 16.8 -> 15.3 mm
- net /esp32-c6 Pinout/IO18: track 16.6 -> 15.3 mm
- net /esp32-c6 Pinout/IO20: track 17.8 -> 16.6 mm
Other:
- board text added: "REV A 12/25"
- board text added: "SCL"
- board text added: "SDA"
- board text added: "VCC"
