File: esp32-c6.kicad_sch (KiCad schematic)
At the start: 37 parts, among them J1 USB_C_Receptacle_USB2.0_14P, J2 USB_C_Receptacle_USB2.0_14P, Q1 BC847BDW1, SW1 SW_Push, SW2 SW_Push, U1 CP2102N-Axx-xQFN28

Commit message: Refinement to pcb and schematic layout
Other:
- title: (none) -> ESP32-C6 Dev Board
- moved on the sheet: C1, C2, C3, C4, C5, C6, C7, D1, D13, D14, D2, D3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
